File: Hardware/PreAmp.kicad_sch (KiCad schematic)
At the start: 0 parts

Commit message: Imported OPA1656 into project and library
Parts:
- added U1: OPA1656ID, OPA1656ID:SOIC127P599X175-8N, symbol OPA1656ID:OPA1656ID
