File: Hardware/KiCad/Main_Board/PreAmp.kicad_sch (KiCad schematic)
At the start: 0 parts

Commit message: Added headers and mounting holes for connection with other PCB
Parts:
- added H1, H2, H3, H4: MountingHole_Pad, MountingHole:MountingHole_3.2mm_M3_DIN965_Pad_TopBottom, symbol Mechanical:MountingHole_Pad
- added J7: Conn_01x05_Socket, symbol Connector:Conn_01x05_Socket
Connections:
- new net +5V: J7.5 (Pin_5)
- new net 5V-: J7.3 (Pin_3)
- new net GND: H1.1, H2.1, H3.1, H4.1, J7.2 (Pin_2), J7.4 (Pin_4)
- new net MIC_OUT: J7.1 (Pin_1)
Other:
- note added: "Female Header to Preamp PCB"
- note added: "Mounting Holes"
