File: Hardware/KiCad/Main_Board/MCU.kicad_sch (KiCad schematic)
At the start: 5 parts, among them J1 Conn_01x24_FPC, J8 Conn_01x24_FPC, U2 Teensy4.1

Commit message: Interface hierarchical out for screen and encoder
Parts:
- renumbered J1 to J?, TP(D+) to TP(D+)?, U2 to U?
Connections:
- net D+: no longer TP(D-).1
- new net D-: TP(D-).1
Changed lines of the file:
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@@
+		)
+	)
+	(global_label "3.3V"
+		(shape output)
+		(at 106.68 105.41 180)
+		(fields_autoplaced yes)
+		(effects
+			(font
+				(size 1.27 1.27)
+			)
+			(justify right)
+		)
+		(property "Intersheetrefs" "${INTERSHEET_REFS}"
+			(at 99.5824 105.41 0)
+			(effects
+				(font
+					(size 1.27 1.27)
+				)
+				(justify right)
+				(hide yes)
+			)
 		)
 	)
@@
 		)
 	)
-	(hierarchical_label "3.3V"
-		(shape output)
-		(at 106.68 105.41 180)
-		(effects
-			(font
-				(size 1.27 1.27)
-			)
-			(justify right)
-		)
-	)
 	(hierarchical_label "40"
 		(shape output)
@@
 		)
 	)
-	(hierarchical_label "D+"
+	(hierarchical_label "D-"
 		(shape input)
 		(at 106.68 143.51 180)
@@
 		(on_board yes)
 		(dnp no)
-		(property "Reference" "J1"
+		(property "Reference" "J?"
 			(at 190.5 67.056 0)
 			(effects
@@
 		)
 		(pin "7"
+		)
+		(instances
+			(project "Main_Board"
+				(path "/e827c80a-ca8d-4d24-8db6-878b575a1aed/80744173-9491-4551-a74b-98f5922bdb3a"
+					(reference "J?")
+					(unit 1)
+				)
+			)
 		)
 	)
@@
 		(on_board yes)
 		(dnp no)
-		(property "Reference" "TP(D+)"
+		(property "Reference" "TP(D+)?"
 			(at 114.046 139.7 90)
 			(effects
@@
 		)
 		(pin "1"
+		)
+		(instances
+			(project "Main_Board"
+				(path "/e827c80a-ca8d-4d24-8db6-878b575a1aed/80744173-9491-4551-a74b-98f5922bdb3a"
+					(reference "TP(D+)?")
+					(unit 1)
+				)
+			)
 		)
 	)
@@
 		(dnp no)
 		(fields_autoplaced yes)
-		(property "Reference" "U2"
+		(property "Reference" "U?"
 			(at 152.4 58.42 0)
 			(effects
@@
 		(pin "66"
 		)
-	)
+		(instances
+			(project "Main_Board"
+				(path "/e827c80a-ca8d-4d24-8db6-878b575a1aed/80744173-9491-4551-a74b-98f5922bdb3a"
+					(reference "U?")
+					(unit 1)
+				)
+			)
+		)
+	)

Commit message: Screen pinout for MCU
Connections:
- net 26 renamed 26(SDA)
- net 27 renamed 27(SCL)
- net 28 renamed 28(RST)
- net 29 renamed 29(DC)
- net 30 renamed 30(CS)
- net 33 renamed 33(PinA)
- net 34 renamed 34(PinB)
- net 35 renamed 35(ENC_BTN)
Changed lines of the file:
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@@
 		)
 	)
-	(hierarchical_label "33"
+	(hierarchical_label "33(PinA)"
 		(shape output)
 		(at 200.66 128.27 0)
@@
 		)
 	)
-	(hierarchical_label "26"
+	(hierarchical_label "26(SDA)"
 		(shape output)
 		(at 106.68 113.03 180)
@@
 		)
 	)
-	(hierarchical_label "29"
+	(hierarchical_label "29(DC)"
 		(shape output)
 		(at 106.68 120.65 180)
@@
 		)
 	)
-	(hierarchical_label "35"
+	(hierarchical_label "35(ENC_BTN)"
 		(shape output)
 		(at 200.66 123.19 0)
@@
 		)
 	)
-	(hierarchical_label "27"
+	(hierarchical_label "27(SCL)"
 		(shape output)
 		(at 106.68 115.57 180)
@@
 		)
 	)
-	(hierarchical_label "30"
+	(hierarchical_label "30(CS)"
 		(shape output)
 		(at 106.68 123.19 180)
@@
 		)
 	)
-	(hierarchical_label "28"
+	(hierarchical_label "28(RST)"
 		(shape output)
 		(at 106.68 118.11 180)
@@
 		)
 	)
-	(hierarchical_label "34"
+	(hierarchical_label "34(PinB)"
 		(shape output)
 		(at 200.66 125.73 0)
